Commit message: Generate visual meshes for the humanoid approximation
Replace the primitive visuals with procedurally generated geometry, keeping
convex primitives for collision.

- meshes.py: lofted superellipse sections build tapered limb segments with
  chamfered ends, cylindrical actuator housings straddling each joint, a
  pinched trunk, and a forward-facing disc head. Shapes follow published
  descriptions of the robot's design language, not any third-party model
- build_eatlas.py writes one OBJ per link and points the URDF's <visual> at
  them; <collision> keeps the convex primitive, so contact cost is unchanged
  no matter how detailed the visual gets
- the viewer now renders the exported mesh directly, so it cannot drift from
  what the OBJ files contain

13 mesh tests, including a directed-edge check that catches unclosed shells
and inconsistent winding in one pass, bounds that must stay inside the
collider they stand in for, and a face budget ceiling. 1348 faces total.

A stock marketplace model was considered and rejected: the licence forbids
redistribution and warns of third-party trademark, and a single unarticulated
shell cannot drive a URDF without being cut into links by hand anyway. The
reasoning is recorded in docs/asset-notes.md.

Co-Authored-By: Claude Opus 5 <noreply@anthropic.com>
Claude-Session: https://claude.ai/code/session_015geVMxpZio7YNQJkjkkqps

File: masonry_rl/assets/eatlas_approx.urdf (robot description, URDF)
Before this commit: robot eatlas_approx, 47 links, 46 joints
Links:
- link head: geometry collision box size=0.180000 0.160000 0.220000; visual mesh filename=meshes/head.obj
- link l_foot: geometry collision box size=0.288800 0.110000 0.074100; visual mesh filename=meshes/l_foot.obj
- link l_forearm: geometry collision cylinder length=0.299947 radius=0.048000; visual mesh filename=meshes/l_forearm.obj
- link l_gripper_0: geometry collision box size=0.020000 0.020000 0.090000; visual mesh filename=meshes/l_gripper_0.obj
- link l_gripper_1: geometry collision box size=0.020000 0.020000 0.090000; visual mesh filename=meshes/l_gripper_1.obj
- link l_hand: geometry collision box size=0.050000 0.090000 0.221879; visual mesh filename=meshes/l_hand.obj
- link l_shank: geometry collision cylinder length=0.467400 radius=0.060000; visual mesh filename=meshes/l_shank.obj
- link l_thigh: geometry collision cylinder length=0.465500 radius=0.075000; visual mesh filename=meshes/l_thigh.obj
- link l_upper_arm: geometry collision cylinder length=0.382124 radius=0.055000; visual mesh filename=meshes/l_upper_arm.obj
- link pelvis: geometry collision box size=0.220000 0.362900 0.160000; visual mesh filename=meshes/pelvis.obj
- link r_foot: geometry collision box size=0.288800 0.110000 0.074100; visual mesh filename=meshes/r_foot.obj
- link r_forearm: geometry collision cylinder length=0.299947 radius=0.048000; visual mesh filename=meshes/r_forearm.obj
- link r_gripper_0: geometry collision box size=0.020000 0.020000 0.090000; visual mesh filename=meshes/r_gripper_0.obj
- link r_gripper_1: geometry collision box size=0.020000 0.020000 0.090000; visual mesh filename=meshes/r_gripper_1.obj
- link r_hand: geometry collision box size=0.050000 0.090000 0.221879; visual mesh filename=meshes/r_hand.obj
- link r_shank: geometry collision cylinder length=0.467400 radius=0.060000; visual mesh filename=meshes/r_shank.obj
- link r_thigh: geometry collision cylinder length=0.465500 radius=0.075000; visual mesh filename=meshes/r_thigh.obj
- link r_upper_arm: geometry collision cylinder length=0.382124 radius=0.055000; visual mesh filename=meshes/r_upper_arm.obj
- link torso: geometry collision box size=0.240000 0.320000 0.475824; visual mesh filename=meshes/torso.obj
